Commit message: Testing

File: ca_description/urdf/sensors/lasers/rplidar.xacro (robot description, xacro)
@@ -15,5 +15,6 @@
 <xacro:property name="topic_name"    value="${name}/scan"/>
 <joint name="${name}_joint" type="fixed">
-  <origin xyz="${laser_origin}"/>
+  <!-- https://www.seeedstudio.com/blog/2018/11/09/rplidar-and-ros-the-best-way-to-learn-robot-and-slam/ -->
+  <origin xyz="${laser_origin}" rpy="0 0 ${pi}"/>
   <parent link="${parent_link}"/>
   <child link="${link_name}"/>

File: ca_description/urdf/stacks/turtlebot.xacro (robot description, xacro)
@@ -10,5 +10,5 @@
   <joint name="pole_${name}_joint" type="fixed">
     <xacro:insert_block name="origin"/>
-    <parent link="${parent}"/>
+    <parent link="${parent}" rpy="0 0 ${pi}"/>
     <child link="${link_name}"/>
   </joint>
